File: rev4/rp2040-memcard.kicad_pcb (KiCad board)
At the start: 2 copper layers, 35.9 x 62.7 mm, 60 parts, among them J1 PSX-Memcard, J18 G, J19 3V3, J2 OLED, J3 USB_C_Receptacle_USB2.0, J4 +, J5 D, J6 C, J7 G, J8 TX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

Commit message: finalize rev4
Parts:
- SW1, SW2: footprint kicad_lceda:SW-SMD_TS24CA -> kicad_lceda:SW-TH_TSC017A10026A; moved to B.Cu
- SW3: footprint kicad_lceda:SW-SMD_TS24CA -> Connector_PinHeader_2.00mm:PinHeader_1x02_P2.00mm_Vertical
- moved R3 6.54 mm to (54.4, 48.0)
- moved R4 6.54 mm to (55.4, 48.0)
- moved SW3 2.35 mm to (48.8, 37.6), turned to 0 degrees
- moved SW1 1.58 mm to (73.0, 29.8)
- moved SW2 1.58 mm to (48.6, 29.8)
Connections:
- SW1 pad 1: unconnected-(SW1-Pad1) -> SW1
- SW1 pad 2: unconnected-(SW1-Pad2) -> GND
- SW1 pad 3: SW1 -> unconnected-(SW1-Pad3)
- SW2 pad 1: unconnected-(SW2-Pad1) -> GND
- SW2 pad 2: unconnected-(SW2-Pad2) -> SW2
- SW2 pad 3: GND -> unconnected-(SW2-Pad3)
- SW3 pad 1: unconnected-(SW3-Pad1) -> GND
- SW3 pad 2: unconnected-(SW3-Pad2) -> Net-(R1-Pad2)
Routing:
- net Net-(R4-Pad2): track 4.97 -> 11.5 mm
- net D+: track 24.8 -> 18.3 mm
- net Net-(R3-Pad2): track 5.23 -> 11.8 mm
- net D-: track 24.8 -> 18.3 mm
- net GND: track 63.4 -> 60.0 mm, vias 31 -> 28
- net Net-(R1-Pad2): track 1.88 -> 4.13 mm
- net SW2: track 69.3 -> 67.8 mm, vias 2 -> 1
- net SW1: track 53.4 -> 52.6 mm, vias 2 -> 1
Other:
- outline, holes or cut-outs redrawn
- board text added: "rev4"
- board text added: "sd2psx"
