File: rev4/rp2040-memcard.kicad_sch (KiCad schematic)
At the start: 60 parts, among them J1 PSX-Memcard, J18 G, J19 3V3, J2 OLED, J3 USB_C_Receptacle_USB2.0, J4 +, J5 D, J6 C, J7 G, J8 TX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

Commit message: finalize rev4
Parts:
- SW1, SW2: footprint kicad_lceda:SW-SMD_TS24CA -> kicad_lceda:SW-TH_TSC017A10026A; symbol kicad_lceda:TS24CA -> kicad_lceda:TSC017A10026A; LCSC C393942 -> (none); SuppliersPartNumber C393942 -> C2888536; uuid std:011ee46cdc964900a13c320feaf84dfd -> std:f38194a8eae74192a85d00db3df68d9a
- SW3: footprint kicad_lceda:SW-SMD_TS24CA -> Connector_PinHeader_2.00mm:PinHeader_1x02_P2.00mm_Vertical; symbol kicad_lceda:TS24CA -> Switch:SW_Push
Connections:
- net GND: now also SW1.2, SW2.1, SW3.1; no longer SW1.4, SW2.3, SW3.3
- net SW1: now also SW1.1; no longer SW1.3
- net SW2: now also SW2.2; no longer SW2.4
- net at SW3.2: now also R1.2
- no-connect marks 23 -> 19

Commit message: remove boot button
Parts:
- SW3: LCSC C393942 -> (none); SuppliersPartNumber C393942 -> (none)
Changed lines of the file:
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@@
       (effects (font (size 1.27 1.27)) hide)
     )
-    (property "SuppliersPartNumber" "C393942" (id 4) (at 40.64 186.69 0)
+    (property "SuppliersPartNumber" "" (id 4) (at 40.64 186.69 0)
       (effects (font (size 1.27 1.27)) hide)
     )
@@
       (effects (font (size 1.27 1.27)) hide)
     )
-    (property "LCSC" "C393942" (id 6) (at 40.64 179.07 0)
+    (property "LCSC" "" (id 6) (at 40.64 179.07 0)
       (effects (font (size 1.27 1.27)) hide)
     )
